File: cad/proto88_new/aarghweeno_88.kicad_pcb (KiCad board)
At the start: 2 copper layers, 99.1 x 99.1 mm, 47 parts, among them J1 Screw_Terminal_01x02, J10 Conn_01x38_Male, J11 Conn_01x38_Male, J12 Conn_01x38_Male, J13 Conn_01x38_Male, J14 Conn_01x38_Male, J15 Conn_01x38_Male, J16 Conn_01x38_Male, J17 Conn_01x38_Male, J18 Conn_01x38_Male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

Commit message: Release Candidate 1 ver 1.0
Parts:
- added G***: LOGO, bdk_art:ste_logo, F.Cu at (163.2, 141.0)
Other:
- board text added: "AVR ATMega 8 / 88 / 168 / 328 Prototype Board Ver. 1.0 Copyright (c) 2022 William R Cooke, Small Time Electronics www.smalltimeelectronics.com"

Commit message: Changed reg cap value, changed version, added port# to LED, cleaned up silkscreen.
Parts:
- C3: value .33 -> 0.1
Other:
- board text added: "AVR ATMega 8 / 88 / 168 / 328 Prototype Board Ver. 1.1 Copyright (c) 2022 William R Cooke, Small Time Electronics www.smalltimeelectronics.com"
- board text removed: "AVR ATMega 8 / 88 / 168 / 328 Prototype Board Ver. 1.0 Copyright (c) 2022 William R Cooke, Small Time Electronics www.smalltimeelectronics.com"
